File: Xbox one shunt.kicad_sch (KiCad schematic)
At the start: 10 parts, among them U2 TLV3201AIDBVR

Commit message: fixed shunt value and resistor value
Parts:
- R1: value 12kΩ -> 10kΩ
- R3: value R_Shunt 0.5Ω -> R_Shunt 2.2Ω
Changed lines of the file:
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@@
 			)
 		)
-		(property "Value" "R_Shunt 0.5Ω"
+		(property "Value" "R_Shunt 2.2Ω"
 			(at 85.344 101.6 0)
 			(effects
@@
 			)
 		)
-		(property "Value" "12kΩ"
+		(property "Value" "10kΩ"
 			(at 107.95 81.28 90)
 			(effects
